Commit message: Create random collision free trajectory

File: panda_moveit_config/config/panda_arm.xacro (robot description, xacro)
@@ -8,48 +8,49 @@
     <!--SUBGROUPS: Groups can also be formed by referencing to already defined group names-->
     <group name="panda_arm">
-      <chain base_link="panda_link0" tip_link="panda_link8" />
+      <chain base_link="panda_right_link0" tip_link="panda_right_link8" />
     </group>
     <!--GROUP STATES: Purpose: Define a named state for a particular group, in terms of joint values. This is useful to define states like 'folded arms'-->
     <group_state name="ready" group="panda_arm">
-      <joint name="panda_joint1" value="0" />
-      <joint name="panda_joint2" value="-0.785" />
-      <joint name="panda_joint3" value="0" />
-      <joint name="panda_joint4" value="-2.356" />
-      <joint name="panda_joint5" value="0" />
-      <joint name="panda_joint6" value="1.571" />
-      <joint name="panda_joint7" value="0.785" />
+      <joint name="panda_right_joint1" value="0" />
+      <joint name="panda_right_joint2" value="-0.785" />
+      <joint name="panda_right_joint3" value="0" />
+      <joint name="panda_right_joint4" value="-2.356" />
+      <joint name="panda_right_joint5" value="0" />
+      <joint name="panda_right_joint6" value="1.571" />
+      <joint name="panda_right_joint7" value="0.785" />
     </group_state>
     <group_state name="extended" group="panda_arm">
-      <joint name="panda_joint1" value="0" />
-      <joint name="panda_joint2" value="0" />
-      <joint name="panda_joint3" value="0" />
-      <joint name="panda_joint4" value="0" />
-      <joint name="panda_joint5" value="0" />
-      <joint name="panda_joint6" value="0" />
-      <joint name="panda_joint7" value="0.785" />
+      <joint name="panda_right_joint2" value="0" />
+      <joint name="panda_right_joint1" value="0" />
+      <joint name="panda_right_joint3" value="0" />
+      <joint name="panda_right_joint4" value="0" />
+      <joint name="panda_right_joint5" value="0" />
+      <joint name="panda_right_joint6" value="0" />
+      <joint name="panda_right_joint7" value="0.785" />
     </group_state>
     <!--END EFFECTOR: Purpose: Represent information about an end effector.-->
     <!--VIRTUAL JOINT: Purpose: this element defines a virtual joint between a robot link and an external frame of reference (considered fixed with respect to the robot)-->
-    <virtual_joint name="virtual_joint" type="floating" parent_frame="world" child_link="panda_link0" />
+    <virtual_joint name="virtual_joint" type="floating" parent_frame="world" child_link="panda_right_link0" />
     <!--DISABLE COLLISIONS: By default it is assumed that any link of the robot could potentially come into collision with any other link in the robot. This tag disables collision checking between a specified pair of links. -->
-    <disable_collisions link1="panda_link0" link2="panda_link1" reason="Adjacent" />
-    <disable_collisions link1="panda_link0" link2="panda_link2" reason="Never" />
-    <disable_collisions link1="panda_link0" link2="panda_link3" reason="Never" />
-    <disable_collisions link1="panda_link0" link2="panda_link4" reason="Never" />
-    <disable_collisions link1="panda_link1" link2="panda_link2" reason="Adjacent" />
-    <disable_collisions link1="panda_link1" link2="panda_link3" reason="Never" />
-    <disable_collisions link1="panda_link1" link2="panda_link4" reason="Never" />
-    <disable_collisions link1="panda_link2" link2="panda_link3" reason="Adjacent" />
-    <disable_collisions link1="panda_link2" link2="panda_link4" reason="Never" />
-    <disable_collisions link1="panda_link2" link2="panda_link6" reason="Never" />
-    <disable_collisions link1="panda_link3" link2="panda_link4" reason="Adjacent" />
-    <disable_collisions link1="panda_link3" link2="panda_link5" reason="Never" />
-    <disable_collisions link1="panda_link3" link2="panda_link6" reason="Never" />
-    <disable_collisions link1="panda_link3" link2="panda_link7" reason="Never" />
-    <disable_collisions link1="panda_link4" link2="panda_link5" reason="Adjacent" />
-    <disable_collisions link1="panda_link4" link2="panda_link6" reason="Never" />
-    <disable_collisions link1="panda_link4" link2="panda_link7" reason="Never" />
-    <disable_collisions link1="panda_link5" link2="panda_link6" reason="Adjacent" />
-    <disable_collisions link1="panda_link6" link2="panda_link7" reason="Adjacent" />
+    <disable_collisions link1="panda_right_link0" link2="panda_right_link1" reason="Adjacent" />
+    <disable_collisions link1="panda_right_link0" link2="panda_right_link2" reason="Never" />
+    <disable_collisions link1="panda_right_link0" link2="panda_right_link3" reason="Never" />
+    <disable_collisions link1="panda_right_link0" link2="panda_right_link4" reason="Never" />
+    <disable_collisions link1="panda_right_link1" link2="panda_right_link2" reason="Adjacent" />
+    <disable_collisions link1="panda_right_link1" link2="panda_right_link3" reason="Never" />
+    <disable_collisions link1="panda_right_link1" link2="panda_right_link4" reason="Never" />
+    <disable_collisions link1="panda_right_link2" link2="panda_right_link3" reason="Adjacent" />
+    <disable_collisions link1="panda_right_link2" link2="panda_right_link4" reason="Never" />
+    <disable_collisions link1="panda_right_link2" link2="panda_right_link6" reason="Never" />
+    <disable_collisions link1="panda_right_link3" link2="panda_right_link4" reason="Adjacent" />
+    <disable_collisions link1="panda_right_link3" link2="panda_right_link5" reason="Never" />
+    <disable_collisions link1="panda_right_link3" link2="panda_right_link6" reason="Never" />
+    <disable_collisions link1="panda_right_link3" link2="panda_right_link7" reason="Never" />
+    <disable_collisions link1="panda_right_link4" link2="panda_right_link5" reason="Adjacent" />
+    <disable_collisions link1="panda_right_link4" link2="panda_right_link6" reason="Never" />
+    <disable_collisions link1="panda_right_link4" link2="panda_right_link7" reason="Never" />
+    <disable_collisions link1="panda_right_link5" link2="panda_right_link6" reason="Adjacent" />
+    <disable_collisions link1="panda_right_link6" link2="panda_right_link7" reason="Adjacent" />
+    <disable_collisions link1="panda_right_link7" link2="panda_right_link8" reason="Adjacent" />
   </xacro:macro>
 </robot>

File: panda_moveit_config/config/panda_arm_hand.srdf.xacro (robot description, xacro)
@@ -27,37 +27,37 @@
   </group_state>
   <!--END EFFECTOR: Purpose: Represent information about an end effector.-->
-  <end_effector name="hand" parent_link="panda_link8" group="hand" parent_group="panda_arm" />
+  <end_effector name="hand" parent_link="panda_right_link8" group="hand" parent_group="panda_arm" />
   <!--DISABLE COLLISIONS: By default it is assumed that any link of the robot could potentially come into collision with any other link in the robot. This tag disables collision checking between a specified pair of links. -->
     <disable_collisions link1="panda_hand" link2="panda_leftfinger" reason="Adjacent" />
-    <disable_collisions link1="panda_hand" link2="panda_link4" reason="Never" />
-    <disable_collisions link1="panda_hand" link2="panda_link6" reason="Never" />
-    <disable_collisions link1="panda_hand" link2="panda_link7" reason="Default" />
-    <disable_collisions link1="panda_hand" link2="panda_link8" reason="Adjacent" />
+    <disable_collisions link1="panda_hand" link2="panda_right_link4" reason="Never" />
+    <disable_collisions link1="panda_hand" link2="panda_right_link6" reason="Never" />
+    <disable_collisions link1="panda_hand" link2="panda_right_link7" reason="Default" />
+    <disable_collisions link1="panda_hand" link2="panda_right_link8" reason="Adjacent" />
     <disable_collisions link1="panda_hand" link2="panda_rightfinger" reason="Adjacent" />
-    <disable_collisions link1="panda_leftfinger" link2="panda_link4" reason="Never" />
-    <disable_collisions link1="panda_leftfinger" link2="panda_link6" reason="Never" />
-    <disable_collisions link1="panda_leftfinger" link2="panda_link7" reason="Never" />
-    <disable_collisions link1="panda_leftfinger" link2="panda_link8" reason="Never" />
-    <disable_collisions link1="panda_link0" link2="panda_link1" reason="Adjacent" />
-    <disable_collisions link1="panda_link0" link2="panda_link2" reason="Never" />
-    <disable_collisions link1="panda_link0" link2="panda_link3" reason="Never" />
-    <disable_collisions link1="panda_link0" link2="panda_link4" reason="Never" />
-    <disable_collisions link1="panda_link1" link2="panda_link4" reason="Never" />
-    <disable_collisions link1="panda_link2" link2="panda_link3" reason="Adjacent" />
-    <disable_collisions link1="panda_link2" link2="panda_link4" reason="Never" />
-    <disable_collisions link1="panda_link3" link2="panda_link4" reason="Adjacent" />
-    <disable_collisions link1="panda_link3" link2="panda_link6" reason="Never" />
-    <disable_collisions link1="panda_link4" link2="panda_link5" reason="Adjacent" />
-    <disable_collisions link1="panda_link4" link2="panda_link6" reason="Never" />
-    <disable_collisions link1="panda_link4" link2="panda_link7" reason="Never" />
-    <disable_collisions link1="panda_link4" link2="panda_link8" reason="Never" />
-    <disable_collisions link1="panda_link4" link2="panda_rightfinger" reason="Never" />
-    <disable_collisions link1="panda_link5" link2="panda_link6" reason="Adjacent" />
-    <disable_collisions link1="panda_link5" link2="panda_link7" reason="Default" />
-    <disable_collisions link1="panda_link6" link2="panda_link7" reason="Adjacent" />
-    <disable_collisions link1="panda_link6" link2="panda_rightfinger" reason="Never" />
-    <disable_collisions link1="panda_link7" link2="panda_link8" reason="Adjacent" />
-    <disable_collisions link1="panda_link7" link2="panda_rightfinger" reason="Never" />
-    <disable_collisions link1="panda_link8" link2="panda_rightfinger" reason="Never" />
-    <disable_collisions link1="panda_link5" link2="panda_hand" reason="Default" />
+    <disable_collisions link1="panda_leftfinger" link2="panda_right_link4" reason="Never" />
+    <disable_collisions link1="panda_leftfinger" link2="panda_right_link6" reason="Never" />
+    <disable_collisions link1="panda_leftfinger" link2="panda_right_link7" reason="Never" />
+    <disable_collisions link1="panda_leftfinger" link2="panda_right_link8" reason="Never" />
+    <disable_collisions link1="panda_right_link0" link2="panda_right_link1" reason="Adjacent" />
+    <disable_collisions link1="panda_right_link0" link2="panda_right_link2" reason="Never" />
+    <disable_collisions link1="panda_right_link0" link2="panda_right_link3" reason="Never" />
+    <disable_collisions link1="panda_right_link0" link2="panda_right_link4" reason="Never" />
+    <disable_collisions link1="panda_right_link1" link2="panda_right_link4" reason="Never" />
+    <disable_collisions link1="panda_right_link2" link2="panda_right_link3" reason="Adjacent" />
+    <disable_collisions link1="panda_right_link2" link2="panda_right_link4" reason="Never" />
+    <disable_collisions link1="panda_right_link3" link2="panda_right_link4" reason="Adjacent" />
+    <disable_collisions link1="panda_right_link3" link2="panda_right_link6" reason="Never" />
+    <disable_collisions link1="panda_right_link4" link2="panda_right_link5" reason="Adjacent" />
+    <disable_collisions link1="panda_right_link4" link2="panda_right_link6" reason="Never" />
+    <disable_collisions link1="panda_right_link4" link2="panda_right_link7" reason="Never" />
+    <disable_collisions link1="panda_right_link4" link2="panda_right_link8" reason="Never" />
+    <disable_collisions link1="panda_right_link4" link2="panda_rightfinger" reason="Never" />
+    <disable_collisions link1="panda_right_link5" link2="panda_right_link6" reason="Adjacent" />
+    <disable_collisions link1="panda_right_link5" link2="panda_right_link7" reason="Default" />
+    <disable_collisions link1="panda_right_link6" link2="panda_right_link7" reason="Adjacent" />
+    <disable_collisions link1="panda_right_link6" link2="panda_rightfinger" reason="Never" />
+    <disable_collisions link1="panda_right_link7" link2="panda_right_link8" reason="Adjacent" />
+    <disable_collisions link1="panda_right_link7" link2="panda_rightfinger" reason="Never" />
+    <disable_collisions link1="panda_right_link8" link2="panda_rightfinger" reason="Never" />
+    <disable_collisions link1="panda_right_link5" link2="panda_hand" reason="Default" />
 </robot>
